Commit message: WIP: integrate Blender terrain into Gazebo
- add Blender terrain to Gazebo simulation
- update .gitignore
- add partial voxel_downsampler implementation (not working yet)
- terrain is currently classified entirely as obstacles
- autonav pipeline is not yet functional
- collision geometry is working as expected

File: src/rover_description/urdf/stereo_camera.xacro (robot description, xacro)
@@ -129,6 +129,6 @@
     <parent link="chassis"/>
     <child link="camera_link"/>
-    <!-- Lifted slightly to match the new chassis height -->
-    <origin xyz="0.2 0 0.20" rpy="0 0 0"/>
+    <!-- The middle value (pitch) ensures the camera always sees the ground -->
+    <origin xyz="0.2 0 0.1" rpy="0 0.35 0"/>
   </joint>
   <link name="camera_link">
@@ -152,5 +152,5 @@
   <gazebo reference="camera_link">
     <sensor type="camera" name="left_camera">
-      <update_rate>30.0</update_rate>
+      <update_rate>10.0</update_rate>
       <topic>/stereo/left/image_raw</topic>
       <gz_frame_id>left_camera_optical_frame</gz_frame_id>
@@ -172,5 +172,5 @@
   <gazebo reference="camera_link">
     <sensor type="camera" name="right_camera">
-      <update_rate>2.0</update_rate>
+      <update_rate>10.0</update_rate>
       <topic>/stereo/right/image_raw</topic>
       <pose>0 -0.1 0 0 0 0</pose>

Commit message: Purged elevation_mapping, STVL introduced
- added objects to blender file
- relying on STVL for math
- removed global costmap
- IMU bridged to rviz, imitates rover's actual orientation
- issue: rover still moves in rviz if stationary in gazebo

File: src/rover_description/urdf/stereo_camera.xacro (robot description, xacro)
@@ -23,8 +23,17 @@
       <odom_publish_frequency>30</odom_publish_frequency>
       <topic>cmd_vel</topic>
-      <odom_topic>odom_raw</odom_topic> <!-- changed from odom and tf-->
+      <odom_topic>odom_raw</odom_topic>
+      <publish_odom_tf>false</publish_odom_tf> <!-- THE FIX: Mute Gazebo's conflicting TF -->
       <tf_topic>/tf_gazebo</tf_topic>
       <frame_id>odom</frame_id>
       <child_frame_id>chassis</child_frame_id>
+    </plugin>
+  </gazebo>
+  <!-- IMU -->
+  <!-- Enable Gazebo IMU System Plugin -->
+  <gazebo>
+    <plugin
+      filename="gz-sim-imu-system"
+      name="gz::sim::systems::Imu">
     </plugin>
   </gazebo>
@@ -130,5 +139,5 @@
     <child link="camera_link"/>
     <!-- The middle value (pitch) ensures the camera always sees the ground -->
-    <origin xyz="0.2 0 0.1" rpy="0 0.35 0"/>
+    <origin xyz="0.2 0 0.1" rpy="0 0.1 0"/>
   </joint>
   <link name="camera_link">
@@ -158,11 +167,11 @@
         <horizontal_fov>1.3962634</horizontal_fov>
         <image>
-          <width>640</width>
-          <height>480</height>
+          <width>320</width>
+          <height>240</height>
           <format>R8G8B8</format>
         </image>
         <clip>
           <near>0.1</near>
-          <far>10.0</far>
+          <far>20</far>
         </clip>
       </camera>
@@ -179,11 +188,11 @@
         <horizontal_fov>1.3962634</horizontal_fov>
         <image>
-          <width>640</width>
-          <height>480</height>
+          <width>320</width>
+          <height>240</height>
           <format>R8G8B8</format>
         </image>
         <clip>
           <near>0.1</near>
-          <far>10.0</far>
+          <far>20</far>
         </clip>
       </camera>

Commit message: feat: flatter terrain, rover mechanics, pointcloud generation

File: src/rover_description/urdf/stereo_camera.xacro (robot description, xacro)
@@ -24,5 +24,5 @@
       <topic>cmd_vel</topic>
       <odom_topic>odom_raw</odom_topic>
-      <publish_odom_tf>false</publish_odom_tf> <!-- THE FIX: Mute Gazebo's conflicting TF -->
+      <publish_odom_tf>false</publish_odom_tf> <!-- Mute Gazebo's conflicting TF -->
       <tf_topic>/tf_gazebo</tf_topic>
       <frame_id>odom</frame_id>
@@ -31,5 +31,4 @@
   </gazebo>
   <!-- IMU -->
-  <!-- Enable Gazebo IMU System Plugin -->
   <gazebo>
     <plugin
@@ -41,16 +40,14 @@
   <!-- BASE CHASSIS & CASTER                      -->
   <!-- ========================================== -->
-  <!-- Chassis Link (Shifted up to accommodate wheels) -->
   <link name="chassis">
     <inertial>
       <mass value="2.0"/>
-      <!-- Shifted center of mass up -->
-      <origin xyz="0 0 0.12" rpy="0 0 0"/>
+      <origin xyz="0 0 0.06" rpy="0 0 0"/>
       <inertia ixx="0.01" ixy="0.0" ixz="0.0" iyy="0.01" iyz="0.0" izz="0.01"/>
     </inertial>
     <visual>
-      <origin xyz="0 0 0.12" rpy="0 0 0"/>
-      <geometry>
-        <box size="0.4 0.3 0.1"/>
+      <origin xyz="0 0 0.06" rpy="0 0 0"/>
+      <geometry>
+        <box size="0.4 0.3 0.08"/>
       </geometry>
       <material name="blue">
@@ -59,7 +56,7 @@
     </visual>
     <collision>
-      <origin xyz="0 0 0.12" rpy="0 0 0"/>
-      <geometry>
-        <box size="0.4 0.3 0.1"/>
+      <origin xyz="0 0 0.1" rpy="0 0 0"/>
+      <geometry>
+        <box size="0.3 0.2 0.02"/>
       </geometry>
     </collision>
@@ -69,10 +66,10 @@
     <parent link="chassis"/>
     <child link="caster_link"/>
-    <origin xyz="-0.15 0 0.04" rpy="0 0 0"/>
+    <origin xyz="-0.15 0 0.02" rpy="0 0 0"/>
   </joint>
   <link name="caster_link">
     <visual>
       <geometry>
-        <sphere radius="0.04"/>
+        <sphere radius="0.02"/>
       </geometry>
       <material name="dark_grey">
@@ -82,5 +79,5 @@
     <collision>
       <geometry>
-        <sphere radius="0.04"/>
+        <sphere radius="0.02"/>
       </geometry>
     </collision>
@@ -90,5 +87,4 @@
     </inertial>
   </link>
-  <!-- Remove friction from the caster so it glides smoothly -->
   <gazebo reference="caster_link">
     <mu1>0.001</mu1>
@@ -103,5 +99,5 @@
         <origin xyz="0 0 0" rpy="1.5708 0 0"/>
         <geometry>
-          <cylinder radius="0.08" length="0.04"/>
+          <cylinder radius="0.06" length="0.04"/>
         </geometry>
         <material name="black">
@@ -112,5 +108,5 @@
         <origin xyz="0 0 0" rpy="1.5708 0 0"/>
         <geometry>
-          <cylinder radius="0.08" length="0.04"/>
+          <cylinder radius="0.06" length="0.04"/>
         </geometry>
       </collision>
@@ -124,6 +120,5 @@
       <parent link="chassis"/>
       <child link="${prefix}_wheel"/>
-      <!-- Wheels mounted forward and out to the sides -->
-      <origin xyz="0.1 ${y_reflect * 0.17} 0.08" rpy="0 0 0"/>
+      <origin xyz="0.1 ${y_reflect * 0.17} 0.06" rpy="0 0 0"/>
       <axis xyz="0 1 0"/>
     </joint>
@@ -134,12 +129,16 @@
   <!-- STEREO CAMERAS                             -->
   <!-- ========================================== -->
-  <!-- Camera Joint & Link -->
   <joint name="camera_joint" type="fixed">
-    <parent link="chassis"/>
-    <child link="camera_link"/>
-    <!-- The middle value (pitch) ensures the camera always sees the ground -->
-    <origin xyz="0.2 0 0.1" rpy="0 0.1 0"/>
-  </joint>
+  <parent link="chassis"/>
+  <child link="camera_link"/>
+  <!-- Pitch down by 0.35 radians (~20 degrees) -->
+  <origin xyz="0.2 0 0.06" rpy="0 0.1 0"/>
+</joint>
   <link name="camera_link">
+    <inertial>
+      <mass value="0.05"/>
+      <origin xyz="0 0 0" rpy="0 0 0"/>
+      <inertia ixx="0.0001" ixy="0" ixz="0" iyy="0.0001" iyz="0" izz="0.0001"/>
+    </inertial>
     <visual>
       <geometry>
@@ -151,6 +150,6 @@
     </visual>
   </link>
-  <!-- Optical Frame -->
-  <joint name="camera_optical_joint" type="fixed">
+  <!-- Left Camera Optical Frame -->
+  <joint name="left_camera_optical_joint" type="fixed">
     <parent link="camera_link"/>
     <child link="left_camera_optical_frame"/>
@@ -158,4 +157,11 @@
   </joint>
   <link name="left_camera_optical_frame"/>
+  <!-- Right Camera Optical Frame (100mm Y-offset matching Gazebo pose) -->
+  <joint name="right_camera_optical_joint" type="fixed">
+    <parent link="camera_link"/>
+    <child link="right_camera_optical_frame"/>
+    <origin xyz="0 -0.1 0" rpy="-1.5708 0 -1.5708"/>
+  </joint>
+  <link name="right_camera_optical_frame"/>
   <!-- Left Camera Sensor -->
   <gazebo reference="camera_link">
@@ -167,11 +173,11 @@
         <horizontal_fov>1.3962634</horizontal_fov>
         <image>
-          <width>320</width>
-          <height>240</height>
+          <width>640</width>
+          <height>480</height>
           <format>R8G8B8</format>
         </image>
         <clip>
           <near>0.1</near>
-          <far>20</far>
+          <far>1</far>
         </clip>
       </camera>
@@ -184,15 +190,15 @@
       <topic>/stereo/right/image_raw</topic>
       <pose>0 -0.1 0 0 0 0</pose>
-      <gz_frame_id>left_camera_optical_frame</gz_frame_id>
+      <gz_frame_id>right_camera_optical_frame</gz_frame_id>
       <camera name="right">
         <horizontal_fov>1.3962634</horizontal_fov>
         <image>
-          <width>320</width>
-          <height>240</height>
+          <width>640</width>
+          <height>480</height>
           <format>R8G8B8</format>
         </image>
         <clip>
           <near>0.1</near>
-          <far>20</far>
+          <far>1</far>
         </clip>
       </camera>

Commit message: Feat: Increased speed, Fixed bridge, added ros_gz_image

File: src/rover_description/urdf/stereo_camera.xacro (robot description, xacro)
@@ -22,6 +22,6 @@
       <wheel_radius>0.08</wheel_radius>
       <odom_publish_frequency>30</odom_publish_frequency>
-      <topic>cmd_vel</topic>
-      <odom_topic>odom_raw</odom_topic>
+      <topic>/cmd_vel</topic>
+      <odom_topic>/odom_raw</odom_topic>
       <publish_odom_tf>false</publish_odom_tf> <!-- Mute Gazebo's conflicting TF -->
       <tf_topic>/tf_gazebo</tf_topic>
@@ -133,5 +133,5 @@
   <child link="camera_link"/>
   <!-- Pitch down by 0.35 radians (~20 degrees) -->
-  <origin xyz="0.2 0 0.06" rpy="0 0.1 0"/>
+  <origin xyz="0.2 0 0.15" rpy="0 0.35 0"/>
 </joint>
   <link name="camera_link">
@@ -171,5 +171,5 @@
       <gz_frame_id>left_camera_optical_frame</gz_frame_id>
       <camera name="left">
-        <horizontal_fov>1.3962634</horizontal_fov>
+        <horizontal_fov>1.74</horizontal_fov>
         <image>
           <width>640</width>
@@ -179,5 +179,5 @@
         <clip>
           <near>0.1</near>
-          <far>1</far>
+          <far>10.0</far>
         </clip>
       </camera>
@@ -192,5 +192,5 @@
       <gz_frame_id>right_camera_optical_frame</gz_frame_id>
       <camera name="right">
-        <horizontal_fov>1.3962634</horizontal_fov>
+        <horizontal_fov>1.74</horizontal_fov>
         <image>
           <width>640</width>
@@ -200,5 +200,5 @@
         <clip>
           <near>0.1</near>
-          <far>1</far>
+          <far>10.0</far>
         </clip>
       </camera>
